Commit message: 2023-08-08

File: src/mycobot_description/urdf/600_urdf/mycobot_600_urdf.urdf (robot description, URDF)
Before this commit: robot firefighter, 7 links, 6 joints
Links:
- added link ${ns}link7; collision mesh filename=package://jxz/meshes/base_link.STL; visual mesh filename=package://jxz/meshes/base_link.STL
Joints:
- added joint {ns}output_joint6: type fixed, parent ${ns}link6, child ${ns}link7, origin xyz=-0.025 0.09 -0.02 rpy=0 -1.57 0, axis 0 0 0
